File: AlienDetector_hw/AlienDetector.kicad_pcb (KiCad board)
At the start: 2 copper layers, 57 x 85 mm, 57 parts, among them SW1 SWITCH_H, SW2 BUTTON, SW3 BUTTON, SW4 BUTTON, SW5 BUTTON

Commit message: Proceeding with layout
Parts:
- SW2, SW3, SW4, SW5: footprint BtnsSwitches:BTN_6x6_4x4 -> BtnsSwitches:BTN_4x4_SMD
- moved RP2 61.5 mm to (167.5, 55.5)
- moved RP1 52.5 mm to (114.5, 124.0)
- moved XL2 48.4 mm to (133.5, 90.6), turned to 180 degrees
- moved Logo1 18.9 mm to (142.0, 58.2)
- moved XL3 7.02 mm to (117.0, 60.0)
- moved HOLE1 7.00 mm to (115.5, 51.0)
- moved HOLE2 7.00 mm to (166.5, 51.0)
- turned SW2 to 90 degrees
- turned SW3 to 90 degrees
- turned SW4 to 180 degrees
- turned SW5 to 180 degrees
Other:
- board size 57 x 85 mm -> 57 x 78 mm

Commit message: v2 layout done
Parts:
- removed SW2, SW3, SW4, SW5: BUTTON, BtnsSwitches:BTN_4x4_SMD
- added C27: 220pF, Capacitors:CAP_0603, B.Cu at (160.4, 66.4)
- added C28: 1.8pF, Capacitors:CAP_0402, B.Cu at (152.9, 56.6)
- added C29: 1.5pF, Capacitors:CAP_0402, B.Cu at (156.3, 55.6)
- added C30: 10u, Capacitors:CAP_0603, B.Cu at (147.8, 70.4)
- added C31: 10u, Capacitors:CAP_0603, B.Cu at (147.6, 55.6)
- added C32: 0.1u, Capacitors:CAP_0603, B.Cu at (147.8, 72.0)
- added C33: 0.1u, Capacitors:CAP_0603, B.Cu at (147.6, 57.2)
- added C34: 0.1u, Capacitors:CAP_0603, B.Cu at (147.8, 73.6)
- added C35: 1u, Capacitors:CAP_0603, B.Cu at (137.8, 57.0)
- added C36: 0.1u, Capacitors:CAP_0603, B.Cu at (137.8, 58.6)
- added DD3: CC2500, QFN_DFN:QFN20, B.Cu at (154.8, 65.2)
- added DD4: STMPE811, QFN_DFN:QFN16_4x4_H, B.Cu at (142.8, 57.4)
- added L5: 1.2nH, Inductors:IND_0402, B.Cu at (154.6, 56.1)
- added L6: BLM15AG102, Inductors:IND_0402, B.Cu at (138.6, 60.6)
- added Q1: MMBT2222, SOT:SOT23-3, B.Cu at (140.4, 100.0)
- added R10: 10k, Resistors:RES_0603, B.Cu at (147.6, 59.4)
- added R5: 56k, Resistors:RES_0603, B.Cu at (160.4, 64.8)
- added R6: 100R, Resistors:RES_0603, B.Cu at (149.2, 93.0)
- added R7: 100R, Resistors:RES_0603, B.Cu at (149.2, 91.4)
- added R8: 100R, Resistors:RES_0603, B.Cu at (149.2, 89.8)
- added R9: 100R, Resistors:RES_0603, B.Cu at (149.2, 88.2)
- added U1: ER-TFT024, Connectors:ER-CON50HT-1, B.Cu at (144.3, 79.6)
- BZ1, C10, C19, C2, C24, C3, C4, C8, D1, DA1, L3, L4, Logo1, TP1, XTAL1: moved to B.Cu
- C1, C5: value 0.1u -> 10u; moved to B.Cu
- C11, C7: value 10u -> 1u; moved to B.Cu
- C12: value 18pF -> 0.1u; moved to B.Cu
- C13: value 18pF -> 10u; moved to B.Cu
- C14, C16: value 0.1u -> 18pF; moved to B.Cu
- C15: value 220pF -> 0.1u; moved to B.Cu
- C17: value 100pF -> 0.1u; footprint Capacitors:CAP_0402 -> Capacitors:CAP_0603; moved to B.Cu
- C18: value 100pF -> 220pF; footprint Capacitors:CAP_0402 -> Capacitors:CAP_0603; moved to B.Cu
- C20: value 1pF -> 100pF; moved to B.Cu
- C21: value 220pF -> 100pF; footprint Capacitors:CAP_0603 -> Capacitors:CAP_0402; moved to B.Cu
- C22: value 1pF -> 0.1u; footprint Capacitors:CAP_0402 -> Capacitors:CAP_0603; moved to B.Cu
- C23: value 0.1u -> 1pF; footprint Capacitors:CAP_0603 -> Capacitors:CAP_0402; moved to B.Cu
- C25: value 1.8pF -> 1pF; moved to B.Cu
- C26: value 1.5pF -> 0.1u; footprint Capacitors:CAP_0402 -> Capacitors:CAP_0603; moved to B.Cu
- C6: value 10u -> 0.1u; moved to B.Cu
- C9: value 1u -> 0.1u; moved to B.Cu
- DD1: value STM32F072CxTx -> STM32L476Rx; footprint LQFP_TQFP:LQFP48 -> LQFP_TQFP:LQFP64; moved to B.Cu
- DD2: value CC2500 -> 24C08; footprint QFN_DFN:QFN20 -> SO_DIL_TSSOP:SO8_150MIL; moved to B.Cu
- HOLE1, HOLE2, HOLE3, HOLE4: footprint PCB:Hole2d4_out4d5mm -> PCB:Hole3d3_out5d5mm
- L1: value 22uH -> BLM15AG102; footprint Inductors:IND_1210_LQH32C -> Inductors:IND_0402; moved to B.Cu
- L2: value 1.2nH -> 22uH; footprint Inductors:IND_0402 -> Inductors:IND_1210_LQH32C; moved to B.Cu
- R1, R3: value 100R -> 10k; moved to B.Cu
- R2: value 10k -> 1k; moved to B.Cu
- R4: value 56k -> 10k; moved to B.Cu
- RP1, RP2: footprint PCB:REF_POINT_1MM -> PCB:REF_POINT_2MM; moved to B.Cu
- SW1: footprint BtnsSwitches:SW_SS-12F23 -> BtnsSwitches:SW_SS9
- XL2: value CONN_NOKIA_LCD -> CONN_5; footprint Connectors:NOKIA_10PIN -> Connectors:WB-05(MW-5M); moved to B.Cu
- XL3: value SMA_L -> CONN_3; footprint Connectors:RF_SMA_L -> Connectors:PLS-3
- moved L2 96.7 mm to (147.4, 115.8), turned to 90 degrees
- moved C13 96.2 mm to (158.2, 117.8), turned to 270 degrees
- moved C3 93.8 mm to (147.4, 112.6), turned to 180 degrees
- moved C16 86.3 mm to (147.8, 62.3), turned to 180 degrees
- moved C5 84.9 mm to (147.4, 111.0), turned to 180 degrees
- moved C1 84.1 mm to (161.8, 93.1), turned to 180 degrees
- moved L3 82.2 mm to (157.1, 58.8)
- moved C2 81.6 mm to (162.8, 74.5)
- moved D1 81.4 mm to (152.2, 114.6), turned to 180 degrees
- moved TP1 79.8 mm to (151.0, 68.8)
- moved C9 79.4 mm to (156.4, 86.7)
- moved L4 79.0 mm to (153.8, 58.3), turned to 270 degrees
- moved C19 78.8 mm to (157.5, 60.8)
- moved R2 77.6 mm to (143.4, 100.0), turned to 270 degrees
- moved C18 75.9 mm to (160.4, 63.2)
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Connections:
- BZ1 pad 1: Net-(BZ1-Pad1) -> +3.3V
- BZ1 pad 2: GND -> Net-(BZ1-Pad2)
- C1 pad 1: /LCD_PWR -> GND
- C1 pad 2: GND -> PwrMCU
- C10 pad 1: +3.3V -> GND
- C10 pad 2: GND -> PwrMCU
- C11 pad 1: +3.3V -> GND
- C11 pad 2: GND -> PwrMCU
- C12 pad 1: Net-(C12-Pad1) -> +3.3V
- C13 pad 1: Net-(C13-Pad1) -> +3.3V
- C15 pad 1: +3.3V -> GND
- C15 pad 2: GND -> +3.3V
- C16 pad 1: +3.3V -> Net-(C16-Pad1)
- C17 pad 1: /A1 -> Net-(C17-Pad1)
- C17 pad 2: /A3 -> GND
- C18 pad 1: /A2 -> +3.3V
- C18 pad 2: /A4 -> GND
- C2 pad 1: +3.3V -> GND
- C2 pad 2: GND -> PwrMCU
- C20 pad 1: GND -> /A1
- C21 pad 1: +3.3V -> /A2
- C21 pad 2: GND -> /A4
- C22 pad 1: /A4 -> +3.3V
- C22 pad 2: /A5 -> GND
- C23 pad 1: +3.3V -> GND
- C23 pad 2: GND -> /A3
- C25 pad 1: /A5 -> /A4
- C25 pad 2: GND -> /A5
- C26 pad 1: /RF_Out -> +3.3V
- C3 pad 1: +3.3V -> Net-(C3-Pad1)
- C4 pad 1: Net-(C4-Pad1) -> GND
- C4 pad 2: GND -> PwrMCU
- C5 pad 1: +3.3V -> Net-(C3-Pad1)
- C6 pad 1: Net-(C4-Pad1) -> GND
- C6 pad 2: GND -> PwrMCU
- C7 pad 1: +3.3V -> GND
- C7 pad 2: GND -> PwrMCU
- C8 pad 1: +3.3V -> GND
- C8 pad 2: GND -> PwrMCU
- C9 pad 1: +3.3V -> GND
- C9 pad 2: GND -> PwrMCU
- DD1 pad 1: +3.3V -> PwrMCU
- DD1 pad 10: (no net) -> /TOUCH_INT
- DD1 pad 11: /ADC_BAT -> /LCD_CSX
- DD1 pad 12: (no net) -> GND
- DD1 pad 13: /CC_GDO0 -> PwrMCU
- DD1 pad 14: /CC_CS -> /LCD_TE
- DD1 pad 15: /CC_SCK -> /ADC_BAT
- DD1 pad 16: /CC_MISO -> (no net)
- DD1 pad 17: /CC_MOSI -> /CC_GDO0
- DD1 pad 18: /LCD_PWR -> GND
- DD1 pad 19: (no net) -> PwrMCU
- DD1 pad 20: (no net) -> /CC_CS
- DD1 pad 21: /LCD_SDA -> /CC_SCK
- DD1 pad 22: /LCD_XRES -> /CC_MISO
- DD1 pad 23: GND -> /CC_MOSI
- DD1 pad 24: +3.3V -> /LCD_RD
- DD1 pad 25: /LCD_SCLK -> /LCD_WR
- DD1 pad 26: /LCD_XCS -> /LCD_D0
- DD1 pad 27: /LCD_BCKLT -> /LCD_D1
- DD1 pad 28: (no net) -> /LCD_D2
- DD1 pad 29: (no net) -> /LCD_D10
- DD1 pad 30: /UART_TX -> /LCD_D11
- DD1 pad 31: /UART_RX -> GND
- DD1 pad 32: (no net) -> PwrMCU
- DD1 pad 33: (no net) -> /LCD_D12
- DD1 pad 34: /SWDIO -> /LCD_D13
- DD1 pad 35: GND -> /LCD_D14
- DD1 pad 36: +3.3V -> /LCD_D15
- DD1 pad 37: /SWCLK -> /Buzzer
- DD1 pad 38: (no net) -> Net-(DD1-Pad38)
- DD1 pad 41: Net-(DD1-Pad41) -> (no net)
- DD1 pad 42: Net-(DD1-Pad42) -> /UART_TX
- DD1 pad 43: (no net) -> /UART_RX
- DD1 pad 44: GND -> (no net)
- DD1 pad 46: (no net) -> /SWDIO
- DD1 pad 48: +3.3V -> PwrMCU
- DD1 pad 8: GND -> /SCL
- DD1 pad 9: +3.3V -> /SDA
- DD2 pad 1: /CC_SCK -> GND
- DD2 pad 2: /CC_MISO -> GND
- DD2 pad 3: (no net) -> GND
- DD2 pad 4: +3.3V -> GND
- DD2 pad 5: Net-(C14-Pad1) -> /SDA
- DD2 pad 6: /CC_GDO0 -> /SCL
- DD2 pad 7: /CC_CS -> GND
- DD2 pad 8: Net-(C12-Pad1) -> +3.3V
- L1 pad 1: /Lout -> PwrMCU
- L1 pad 2: Net-(C4-Pad1) -> +3.3V
- L2 pad 1: /A4 -> /Lout
- L2 pad 2: GND -> Net-(C3-Pad1)
- L3 pad 1: /A5 -> /A4
- L3 pad 2: /A3 -> GND
- L4 pad 1: /RF_Out -> /A5
- L4 pad 2: /A5 -> /A3
- R1 pad 1: /LCD_BCKLT -> /ADC_BAT
- R1 pad 2: Net-(R1-Pad2) -> Net-(C3-Pad1)
- R2 pad 1: /ADC_BAT -> Net-(Q1-Pad1)
- R2 pad 2: Net-(C4-Pad1) -> /Buzzer
- R3 pad 1: Net-(BZ1-Pad1) -> +3.3V
- R3 pad 2: (no net) -> /SCL
- R4 pad 1: Net-(DD2-Pad17) -> /SDA
- R4 pad 2: GND -> +3.3V
- SW1 pad 1: Net-(C4-Pad1) -> Net-(C3-Pad1)
- XL2 pad 1: /LCD_SCLK -> GND
- XL2 pad 2: /LCD_SDA -> Net-(DD1-Pad38)
- XL2 pad 3: GND -> Net-(DD1-Pad39)
- XL2 pad 4: /LCD_XCS -> Net-(DD1-Pad40)
- XL2 pad 5: /LCD_XRES -> Net-(DD1-Pad51)
- XTAL1 pad 1: Net-(C12-Pad1) -> Net-(C14-Pad1)
- XTAL1 pad 2: Net-(C13-Pad1) -> Net-(C16-Pad1)
Other:
- board size 57 x 78 mm -> 60 x 76 mm
- net class Default: trace_width 0.25 -> 0.2; via_dia 0.8 -> 0.7; via_drill 0.4 -> 0.3
- net class Wide added: clearance 0.2, trace_width 0.5, via_dia 0.7, via_drill 0.3
- rule pad_to_mask_clearance: 0.2 -> 0.1

Commit message: Proceeding
Parts:
- moved C24 1.02 mm to (150.2, 65.3), turned to 270 degrees
- moved C2 0.80 mm to (162.0, 74.5)
- turned R1 to 270 degrees
Routing:
- net GND: track 0.00 -> 770.7 mm, vias 0 -> 130
- net +3.3V: track 0.00 -> 220.2 mm, vias 0 -> 17
- net PwrMCU: track 0.00 -> 86.0 mm, vias 0 -> 5
- net /SCL: track 0.00 -> 65.6 mm, vias 0 -> 3
- net /SDA: track 0.00 -> 59.6 mm, vias 0 -> 3
- net /TOUCH_INT: track 0.00 -> 38.4 mm, vias 0 -> 2
- net /Buzzer: track 0.00 -> 37.3 mm, vias 0 -> 2
- net /LCD_DC: track 0.00 -> 36.4 mm, vias 0 -> 2
- net /SWCLK: track 0.00 -> 35.7 mm, vias 0 -> 1
- net /SWDIO: track 0.00 -> 33.8 mm, vias 0 -> 1
- net /ADC_BAT: track 0.00 -> 33.4 mm, vias 0 -> 2
- net /UART_RX: track 0.00 -> 31.6 mm, vias 0 -> 1
- net /UART_TX: track 0.00 -> 31.1 mm, vias 0 -> 1
- net Net-(B1-PadA): track 0.00 -> 29.5 mm
- net /LCD_D13: track 0.00 -> 28.6 mm, vias 0 -> 2
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- added copper zone on B.Cu, net GND
- added copper zone on F.Cu, net GND

Commit message: PCB sent to factory
Routing:
- net GND: track 770.7 -> 781.7 mm, vias 130 -> 134
